Commit message: code from 15.03 as is

File: pybullet/simple.urdf (robot description, URDF)
Before this commit: robot pendulum, 4 links, 3 joints
Links:
- added link link_2, mass 0; visual cylinder length=0.5 radius=0.01
- link link_1: geometry visual cylinder length=0.5 radius=0.01
Joints:
- added joint joint_2: type revolute, parent link_1, child link_2, origin xyz=0.0 0 0.5 rpy=0 0 0, axis 0 1 0, limit effort=0 velocity=0
- joint joint_eef: origin xyz=0 0 0.8 rpy=0 0 0 -> xyz=0 0 0.5 rpy=0 0 0; parent link_1 -> link_2

Commit message: fixed two-link robot free motion

File: pybullet/simple.urdf (robot description, URDF)
Before this commit: robot pendulum, 5 links, 4 joints
Links:
- removed link link_eef
- added link link_eef1, mass 1; visual sphere radius=0.05
- added link link_eef2, mass 1; visual sphere radius=0.05
Joints:
- removed joint joint_eef
- added joint joint_eef1: type fixed, parent link_1, child link_eef1, origin xyz=0 0 0.5 rpy=0 0 0
- added joint joint_eef2: type fixed, parent link_2, child link_eef2, origin xyz=0 0 0.5 rpy=0 0 0
- joint joint_2: origin xyz=0.0 0 0.5 rpy=0 0 0 -> xyz=0.0 0 0 rpy=0 0 0; parent link_1 -> link_eef1
